File: 3DPCB Rev B DRV8825.sch (KiCad schematic (older format))
At the start: 192 parts, among them IC1 DRV8825, IC2 DRV8825, IC3 DRV8825, IC4 DRV8825, IC5 DRV8825, J1 SOLDER_JUMPER_3P, J10 , J11 , J12 , J13 , J14 , J15 , J16 , J2 , J3 , J4 , J5 , J6 , J7 , J8 , J9 , K1 CONN_3, K2 CONN_3, K3 CONN_3, K4 CONN_3, K5 CONN_3, K6 CONN_3, K7 CONN_3, P1 CONN_8, P10 CONN_2, P11 CONN_3X2, P12 CONN_3X2, P13 CONN_4, P2 CONN_2, P3 CONN_2, P4 CONN_2, P5 CONN_4, P6 CONN_4, P7 CONN_4, P8 CONN_2, P9 CONN_4, U1 CONN_4_LERCHE, U10 MICRO-SD, U11 TC4427, U12 MCP4728, U13 CONN_4_LERCHE, U15 SPST_MOMENTARY, U16 CONN_4_LERCHE, U17 TC4427, U2 SPST_MOMENTARY, U20 TPS6213X, U21 CONN_4_LERCHE, U22 CONN_4_LERCHE, U23 MCP4728, U24 MOS_NFET, U25 CONN_4_LERCHE, U3 BSS84, U4 CONN_4_LERCHE, U5 MOS_NFET, U6 LPC1768_TQFP100, U7 MOS_NFET, U8 MOS_NFET, U9 CRYSTAL_SMALL

Commit message: Added LercheTech library
Parts:
- C1, C12, C13, C14, C15, C16, C17, C18, C19, C2, C22, C23, C28, C29, C30, C31, C32, C33, C34, C35, C36, C37, C38, C39, C40, C41, C42, C44, C45, C46, C47, C48, C49, C5, C50, C51, C52, C53, C54, C56, C57, C58, C59, C6, C60, C61, C64, C65, C67, C68, C69, C71, C8, C9: symbol C -> C-RESCUE-3DPCB_Rev_B_DRV8825
- C10, C24, C25, C26, C27, C3, C4, C43, C55, C7, C70: symbol CP -> CP-RESCUE-3DPCB_Rev_B_DRV8825
- D1, D2, D3, D4, D6, D7, D8: symbol LED -> LED-RESCUE-3DPCB_Rev_B_DRV8825
- R1, R10, R11, R12, R13, R14, R15, R16, R17, R18, R19, R2, R20, R21, R22, R23, R24, R25, R26, R27, R28, R29, R3, R30, R31, R32, R33, R34, R37, R4, R41, R42, R43, R44, R45, R46, R47, R48, R49, R5, R50, R51, R52, R53, R54, R55, R6, R7, R8, R9: symbol R -> R-RESCUE-3DPCB_Rev_B_DRV8825
